File: CAD/V1.0/ESP-PLC-Relay-Extension-Module-Hardware-Design.kicad_sch (KiCad schematic)
At the start: 32 parts, among them J1 Screw_Terminal_01x04, J2 Conn_01x03_Pin, SW1 SW_DIP_x03, U1 AMS1117-3.3, U2 AOZ1282CI, U3 MCP23017_SO

Commit message: Added Relays
Parts:
- removed D1: M7L, Diode_SMD:D_SMA, symbol Device:D
- removed D2: SMCJ26A, Diode_SMD:D_SMC, symbol Diode:SMCJ26A
- removed SW1: SW_DIP_x03, Button_Switch_THT:SW_DIP_SPSTx03_Slide_9.78x9.8mm_W7.62mm_P2.54mm, symbol Switch:SW_DIP_x03
- added D? (x17): M7L, Diode_SMD:D_SMA, symbol Symbols-Simuncic:M7L
- added D?: SMCJ26A, Diode_SMD:D_SMC, symbol Symbols-Simuncic:SMCJ26A
- added J7 (x4): Screw_Terminal_01x08, Connector_Phoenix_MSTB:PhoenixContact_MSTBA_2,5_8-G-5,08_1x08_P5.08mm_Horizontal, symbol Connector:Screw_Terminal_01x08
- added K1, K? (x15): SJ-10A, Footprints-Simuncic:Relay_SJ-10A, symbol Symbols-Simuncic:SANYOU_SJ-10A
- added Q? (x16): BSS138, Package_TO_SOT_SMD:SOT-23, symbol Transistor_FET:BSS138
- added R? (x16): 200R, Resistor_SMD:R_0603_1608Metric, symbol Device:R
- added R? (x16): 100k, Resistor_SMD:R_0603_1608Metric, symbol Device:R
- added SW?: SW_DIP_x03, Button_Switch_THT:SW_DIP_SPSTx03_Slide_9.78x9.8mm_W7.62mm_P2.54mm, symbol Switch:SW_DIP_x03
Connections:
- net +24V: now also D?.1 (A1), D?.1 (K), D?.1 (K), D?.1 (K), D?.1 (K), D?.1 (K), D?.1 (K), D?.1 (K), D?.1 (K), D?.1 (K), D?.1 (K), D?.1 (K), D?.1 (K), D?.1 (K), D?.1 (K), D?.1 (K), D?.1 (K), D?.1 (K), K1.A2, K?.A2, K?.A2, K?.A2, K?.A2, K?.A2, K?.A2, K?.A2, K?.A2, K?.A2, K?.A2, K?.A2, K?.A2, K?.A2, K?.A2, K?.A2
- net GND: now also D?.2 (A2), Q?.2 (S), Q?.2 (S), Q?.2 (S), Q?.2 (S), Q?.2 (S), Q?.2 (S), Q?.2 (S), Q?.2 (S), Q?.2 (S), Q?.2 (S), Q?.2 (S), Q?.2 (S), Q?.2 (S), Q?.2 (S), Q?.2 (S), Q?.2 (S), R?.2, R?.2, R?.2, R?.2, R?.2, R?.2, R?.2, R?.2, R?.2, R?.2, R?.2, R?.2, R?.2, R?.2, R?.2, R?.2, SW?.4, SW?.5, SW?.6
- net at C3.1, F1.2: now also D?.2 (A)
- net at R7.1, U3.15 (A0): now also SW?.3
- net at R5.1, U3.17 (A2): now also SW?.1
- net at R6.1, U3.16 (A1): now also SW?.2
- net Input0 renamed Relay_0
- net Relay_0: now also R?.1, R?.1
- net Input1 renamed Relay_1
- net Relay_1: now also R?.1, R?.1
- net Input10 renamed Relay_10
- net Relay_10: now also R?.1, R?.1
- net Input11 renamed Relay_11
- net Relay_11: now also R?.1, R?.1
- net Input12 renamed Relay_12
- net Relay_12: now also R?.1, R?.1
- net Input13 renamed Relay_13
- net Relay_13: now also R?.1, R?.1
- net Input14 renamed Relay_14
- net Relay_14: now also R?.1, R?.1
- net Input15 renamed Relay_15
- net Relay_15: now also R?.1, R?.1
- net Input2 renamed Relay_2
- net Relay_2: now also R?.1, R?.1
- net Input3 renamed Relay_3
- net Relay_3: now also R?.1, R?.1
- net Input4 renamed Relay_4
- net Relay_4: now also R?.1, R?.1
- net Input5 renamed Relay_5
- net Relay_5: now also R?.1, R?.1
- net Input6 renamed Relay_6
- net Relay_6: now also R?.1, R?.1
- net Input7 renamed Relay_7
- net Relay_7: now also R?.1, R?.1
- net Input8 renamed Relay_8
- net Relay_8: now also R?.1, R?.1
- net Input9 renamed Relay_9
- net Relay_9: now also R?.1, R?.1
- new net: D?.2 (A), K?.A1, Q?.3 (D) (x15)
- new net: Q?.1 (G), R?.2 (x16)
- new net: D?.2 (A), K1.A1, Q?.3 (D)
- new net Relay_0A: J7.1 (Pin_1), K1.14
- new net Relay_0B: J7.2 (Pin_2), K1.13
- new net Relay_10A: J7.5 (Pin_5), K?.14
- new net Relay_10B: J7.6 (Pin_6), K?.13
- new net Relay_11A: J7.7 (Pin_7), K?.14
- new net Relay_11B: J7.8 (Pin_8), K?.13
- new net Relay_12A: J7.1 (Pin_1), K?.14
- new net Relay_12B: J7.2 (Pin_2), K?.13
- new net Relay_13A: J7.3 (Pin_3), K?.14
- new net Relay_13B: J7.4 (Pin_4), K?.13
- new net Relay_14A: J7.5 (Pin_5), K?.14
- new net Relay_14B: J7.6 (Pin_6), K?.13
- new net Relay_15A: J7.7 (Pin_7), K?.14
- new net Relay_15B: J7.8 (Pin_8), K?.13
- new net Relay_1A: J7.3 (Pin_3), K?.14
- new net Relay_1B: J7.4 (Pin_4), K?.13
- new net Relay_2A: J7.5 (Pin_5), K?.14
- new net Relay_2B: J7.6 (Pin_6), K?.13
- new net Relay_3A: J7.7 (Pin_7), K?.14
- new net Relay_3B: J7.8 (Pin_8), K?.13
- new net Relay_4A: J7.1 (Pin_1), K?.14
- new net Relay_4B: J7.2 (Pin_2), K?.13
- new net Relay_5A: J7.3 (Pin_3), K?.14
- new net Relay_5B: J7.4 (Pin_4), K?.13
- new net Relay_6A: J7.5 (Pin_5), K?.14
- new net Relay_6B: J7.6 (Pin_6), K?.13
- new net Relay_7A: J7.7 (Pin_7), K?.14
- new net Relay_7B: J7.8 (Pin_8), K?.13
- new net Relay_8A: J7.1 (Pin_1), K?.14
- new net Relay_8B: J7.2 (Pin_2), K?.13
- new net Relay_9A: J7.3 (Pin_3), K?.14
- new net Relay_9B: J7.4 (Pin_4), K?.13
Other:
- note added: "16x Digital Output Expander I2C"
- note added: "16x Relay Outputs"
- note added: "Relay Outputs and Connectors"
- note added: "Terminal Blocks for Relay Outputs"
- title: (none) -> ESP-PLC Relay Extension Module
- moved on the sheet: C11, D4, D5, J2, R2, R5, R6, R7, R8, U3

Commit message: PCB designing
Parts:
- removed C1: 10u, Capacitor_SMD:C_0805_2012Metric, symbol Device:C
- removed C4: 22u/50V, Capacitor_THT:CP_Radial_D6.3mm_P2.50mm, symbol Device:C_Polarized
- removed D?: SMCJ26A, Diode_SMD:D_SMC, symbol Symbols-Simuncic:SMCJ26A
- added D10, D11, D12, D13, D18, D19, D20, D21, D26, D27, D28, D29, D34, D35, D36, D37: LED, LED_SMD:LED_0805_2012Metric, symbol Device:LED
- added D2: SMBJ26A, Diode_SMD:D_SMB, symbol Symbols-Simuncic:SMBJ26A
- added R11, R13, R15, R21, R23, R25, R27, R33, R35, R37, R39, R45, R47, R49, R51, R9: 10k, Resistor_SMD:R_0603_1608Metric, symbol Device:R
- J1: footprint Connector_Phoenix_MSTB:PhoenixContact_MSTBA_2,5_4-G-5,08_1x04_P5.08mm_Horizontal -> Connector_Phoenix_MSTB:PhoenixContact_MSTBVA_2,5_4-G-5,08_1x04_P5.08mm_Vertical
- L1: footprint Inductor_SMD:L_FerroCore_HPI1040_10.8x10.0mm -> Footprints-Simuncic:L_FerroCore_HPI1040_10.8x10.0mm
- gave numbers to parts that had none: 81
Connections:
- net +24V: now also D2.1 (A1), R11.1, R13.1, R15.1, R21.1, R23.1, R25.1, R27.1, R33.1, R35.1, R37.1, R39.1, R45.1, R47.1, R49.1, R51.1, R9.1
- net GND: now also D2.2 (A2); no longer D4.1 (K)
- net I2C_SDA: now also D4.1 (K)
- net Relay_0A: now also J7.2 (Pin_2); no longer J7.1 (Pin_1)
- net Relay_0B: now also J7.1 (Pin_1); no longer J7.2 (Pin_2)
- net Relay_10A: now also J7.6 (Pin_6); no longer J7.5 (Pin_5)
- net Relay_10B: now also J7.5 (Pin_5); no longer J7.6 (Pin_6)
- net Relay_11A: now also J7.8 (Pin_8); no longer J7.7 (Pin_7)
- net Relay_11B: now also J7.7 (Pin_7); no longer J7.8 (Pin_8)
- net Relay_12A: now also J7.2 (Pin_2); no longer J7.1 (Pin_1)
- net Relay_12B: now also J7.1 (Pin_1); no longer J7.2 (Pin_2)
- net Relay_13A: now also J7.4 (Pin_4); no longer J7.3 (Pin_3)
- net Relay_13B: now also J7.3 (Pin_3); no longer J7.4 (Pin_4)
- net Relay_14A: now also J7.6 (Pin_6); no longer J7.5 (Pin_5)
- net Relay_14B: now also J7.5 (Pin_5); no longer J7.6 (Pin_6)
- net Relay_15A: now also J7.8 (Pin_8); no longer J7.7 (Pin_7)
- net Relay_15B: now also J7.7 (Pin_7); no longer J7.8 (Pin_8)
- net Relay_1A: now also J7.4 (Pin_4); no longer J7.3 (Pin_3)
- net Relay_1B: now also J7.3 (Pin_3); no longer J7.4 (Pin_4)
- net Relay_2A: now also J7.6 (Pin_6); no longer J7.5 (Pin_5)
- net Relay_2B: now also J7.5 (Pin_5); no longer J7.6 (Pin_6)
- net Relay_3A: now also J7.8 (Pin_8); no longer J7.7 (Pin_7)
- net Relay_3B: now also J7.7 (Pin_7); no longer J7.8 (Pin_8)
- net Relay_4A: now also J7.2 (Pin_2); no longer J7.1 (Pin_1)
- net Relay_4B: now also J7.1 (Pin_1); no longer J7.2 (Pin_2)
- net Relay_5A: now also J7.4 (Pin_4); no longer J7.3 (Pin_3)
- net Relay_5B: now also J7.3 (Pin_3); no longer J7.4 (Pin_4)
- net Relay_6A: now also J7.6 (Pin_6); no longer J7.5 (Pin_5)
- net Relay_6B: now also J7.5 (Pin_5); no longer J7.6 (Pin_6)
- net Relay_7A: now also J7.8 (Pin_8); no longer J7.7 (Pin_7)
- net Relay_7B: now also J7.7 (Pin_7); no longer J7.8 (Pin_8)
- net Relay_8A: now also J7.2 (Pin_2); no longer J7.1 (Pin_1)
- net Relay_8B: now also J7.1 (Pin_1); no longer J7.2 (Pin_2)
- net Relay_9A: now also J7.4 (Pin_4); no longer J7.3 (Pin_3)
- net Relay_9B: now also J7.3 (Pin_3); no longer J7.4 (Pin_4)
- net at D9.2 (A), K4.A1, Q4.3 (D): now also D13.1 (K)
- net at D16.2 (A), K7.A1, Q7.3 (D): now also D20.1 (K)
- net at D31.2 (A), K14.A1, Q14.3 (D): now also D35.1 (K)
- net at D17.2 (A), K8.A1, Q8.3 (D): now also D21.1 (K)
- net at D32.2 (A), K15.A1, Q15.3 (D): now also D36.1 (K)
- net at D23.2 (A), K10.A1, Q10.3 (D): now also D27.1 (K)
- net at D7.2 (A), K2.A1, Q2.3 (D): now also D11.1 (K)
- net at D15.2 (A), K6.A1, Q6.3 (D): now also D19.1 (K)
- net at D33.2 (A), K16.A1, Q16.3 (D): now also D37.1 (K)
- net at D22.2 (A), K9.A1, Q9.3 (D): now also D26.1 (K)
- net at D14.2 (A), K5.A1, Q5.3 (D): now also D18.1 (K)
- net at D6.2 (A), K1.A1, Q1.3 (D): now also D10.1 (K)
- net at D30.2 (A), K13.A1, Q13.3 (D): now also D34.1 (K)
- net at D25.2 (A), K12.A1, Q12.3 (D): now also D29.1 (K)
- net at D8.2 (A), K3.A1, Q3.3 (D): now also D12.1 (K)
- net at D24.2 (A), K11.A1, Q11.3 (D): now also D28.1 (K)
- new net: D36.2 (A), R49.2
- new net: D27.2 (A), R35.2
- new net: D20.2 (A), R25.2
- new net: D10.2 (A), R9.2
- new net: D21.2 (A), R27.2
- new net: D18.2 (A), R21.2
- new net: D11.2 (A), R11.2
- new net: D37.2 (A), R51.2
- new net: D28.2 (A), R37.2
- new net: D12.2 (A), R13.2
- new net: D19.2 (A), R23.2
- new net: D13.2 (A), R15.2
- new net: D34.2 (A), R45.2
- new net: D35.2 (A), R47.2
- new net: D26.2 (A), R33.2
- new net: D29.2 (A), R39.2
Other:
- note added: "230Vac@10A Relay Outputs"
- note added: "Connectors"
- note added: "Digital Output Expander 0-15"
- note added: "I2C Connector with ESD protection"
- note removed: "Digital Input Expander 0-15"
- note removed: "Relay Outputs and Connectors"
- moved on the sheet: C10, C11, C2, C3, C5, C6, C7, C8, C9, D1, D14, D15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
