File: CAD/V1.0/ESP-PLC-Relay-Extension-Module-Hardware-Design.kicad_pcb (KiCad board)
At the start: 2 copper layers, 94 x 100 mm, 146 parts, among them J1 Screw_Terminal_01x04, J2 Conn_01x03_Pin, J3 Screw_Terminal_01x08, J4 Screw_Terminal_01x08, J5 Screw_Terminal_01x08, J6 Screw_Terminal_01x08, K1 SJ-10A, K10 SJ-10A, K11 SJ-10A, K12 SJ-10A, K13 SJ-10A, K14 SJ-10A, K15 SJ-10A, K16 SJ-10A, K2 SJ-10A, K3 SJ-10A, K4 SJ-10A, K5 SJ-10A, K6 SJ-10A, K7 SJ-10A, K8 SJ-10A, K9 SJ-10A, Q1 BSS138, Q10 BSS138, Q11 BSS138, Q12 BSS138, Q13 BSS138, Q14 BSS138, Q15 BSS138, Q16 BSS138, Q2 BSS138, Q3 BSS138, Q4 BSS138, Q5 BSS138, Q6 BSS138, Q7 BSS138, Q8 BSS138, Q9 BSS138, SW1 SW_DIP_x03, U1 AMS1117-3.3, U2 AOZ1282CI, U3 MCP23017_SO

Commit message: PCB Routing
Parts:
- moved J2 5.12 mm to (159.2, 84.5), turned to 90 degrees
- moved D4 5.00 mm to (163.9, 83.8)
- moved R8 4.50 mm to (130.2, 88.7)
- moved D5 3.60 mm to (163.9, 80.2), turned to -90 degrees
- moved R5 1.50 mm to (131.7, 88.7)
- moved R6 1.50 mm to (133.2, 88.7)
- moved R7 1.50 mm to (134.7, 88.7)
- moved C11 0.15 mm to (143.9, 74.5)
- turned R11 to 90 degrees
- turned R13 to -90 degrees
- turned R15 to -90 degrees
- turned R21 to 90 degrees
- turned R23 to 90 degrees
- turned R25 to -90 degrees
- turned R27 to -90 degrees
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Routing:
- net +24V: track 11.3 -> 256.1 mm
- net /Relay_8: track 0.00 -> 48.5 mm
- net /Relay_7: track 2.29 -> 43.2 mm
- net /Relay_9: track 0.00 -> 38.9 mm
- net /Relay_0: track 2.36 -> 40.7 mm
- net /Relay_15: track 0.00 -> 35.2 mm
- net /Relay_6: track 2.36 -> 33.7 mm
- net /Relay_10: track 0.00 -> 29.4 mm
- net /I2C_SDA: track 0.00 -> 28.8 mm
- net /Relay_1: track 2.36 -> 31.0 mm
- net /Relay_14: track 0.00 -> 25.6 mm
- net /I2C_SCL: track 0.00 -> 24.3 mm
- net /Relay_5: track 2.37 -> 24.4 mm
- net Net-(U3-~{RESET}): track 0.00 -> 20.5 mm
- net /Relay_11: track 0.00 -> 19.9 mm
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- added copper zone on B.Cu, net GND
- added copper zone on F.Cu, net GND

Commit message: Final Commit, files sent to JLCPCB
Routing:
- net +24V: track 256.1 -> 535.2 mm, vias 3 -> 5
- net +3V3: track 6.10 -> 61.5 mm, vias 1 -> 3
- net GND: track 2.15 -> 5.34 mm, vias 15 -> 170
